File: PCB_Shield_STM32/PCB_Shield_STM32.kicad_sch (KiCad schematic)
At the start: 8 parts, among them CN10 Conn_02x19_Odd_Even, CN11 Conn_01x02, CN12 Conn_01x02, CN5 Conn_01x10, CN6 Conn_01x08, CN7 Conn_02x19_Odd_Even, CN8 Conn_01x06, CN9 Conn_01x08

Commit message: updated pcb.
Parts:
- added Audio_In1: SN49B11, SN49B11:SWITCHCRAFT_SN49B11, symbol SN49B11:SN49B11
- added C1: 680p, Capacitor_THT:C_Axial_L3.8mm_D2.6mm_P7.50mm_Horizontal, symbol Device:C
- added C2, C8: 1n, Capacitor_THT:C_Axial_L3.8mm_D2.6mm_P7.50mm_Horizontal, symbol Device:C
- added C3: 220p, Capacitor_THT:C_Axial_L3.8mm_D2.6mm_P7.50mm_Horizontal, symbol Device:C
- added C4: 1.8n, Capacitor_THT:C_Axial_L3.8mm_D2.6mm_P7.50mm_Horizontal, symbol Device:C
- added C5: 180p, Capacitor_THT:C_Axial_L3.8mm_D2.6mm_P7.50mm_Horizontal, symbol Device:C
- added C6: 270µ, Capacitor_THT:C_Axial_L3.8mm_D2.6mm_P7.50mm_Horizontal, symbol Device:C
- added C7: 150µ, Capacitor_THT:C_Axial_L3.8mm_D2.6mm_P7.50mm_Horizontal, symbol Device:C
- added D1, D2, D3: LED, LED_THT:LED_D3.0mm, symbol Device:LED
- added J1: Barrel_Jack_Switch, Connector_BarrelJack:BarrelJack_Horizontal, symbol Connector:Barrel_Jack_Switch
- added R1, R2, R3, R8, R9: 56K, Resistor_THT:R_Axial_DIN0204_L3.6mm_D1.6mm_P5.08mm_Horizontal, symbol Device:R
- added R10: 800, Resistor_THT:R_Axial_DIN0204_L3.6mm_D1.6mm_P5.08mm_Horizontal, symbol Device:R
- added R11: 4.45K, Resistor_THT:R_Axial_DIN0204_L3.6mm_D1.6mm_P5.08mm_Horizontal, symbol Device:R
- added R12, R6: 1K, Resistor_THT:R_Axial_DIN0204_L3.6mm_D1.6mm_P5.08mm_Horizontal, symbol Device:R
- added R13, R14, R15, R16, R19: 220, Resistor_THT:R_Axial_DIN0204_L3.6mm_D1.6mm_P5.08mm_Horizontal, symbol Device:R
- added R17, R18: 10k, Resistor_THT:R_Axial_DIN0204_L3.6mm_D1.6mm_P5.08mm_Horizontal, symbol Device:R
- added R4: 10K, Resistor_THT:R_Axial_DIN0204_L3.6mm_D1.6mm_P5.08mm_Horizontal, symbol Device:R
- added R5: 31K, Resistor_THT:R_Axial_DIN0204_L3.6mm_D1.6mm_P5.08mm_Horizontal, symbol Device:R
- added R7: 150k, Resistor_THT:R_Axial_DIN0204_L3.6mm_D1.6mm_P5.08mm_Horizontal, symbol Device:R
- added SW1: SW_SPST, Button_Switch_THT:SW_DIP_SPSTx01_Slide_9.78x4.72mm_W7.62mm_P2.54mm, symbol Switch:SW_SPST
- added U1, U2, U3, U4, U6: OP07, OP07DP:DIP794W45P254L959H508Q8, symbol Amplifier_Operational:OP07
- CN10, CN7: footprint (none) -> Connector_PinSocket_2.54mm:PinSocket_2x19_P2.54mm_Vertical
- CN11, CN12: footprint (none) -> Connector_PinSocket_2.54mm:PinSocket_1x02_P2.54mm_Vertical
- CN5: footprint (none) -> Connector_PinSocket_2.54mm:PinSocket_1x10_P2.54mm_Vertical
- CN6, CN9: footprint (none) -> Connector_PinSocket_2.54mm:PinSocket_1x08_P2.54mm_Vertical
- CN8: footprint (none) -> Connector_PinSocket_2.54mm:PinSocket_1x06_P2.54mm_Vertical
Connections:
- net PA13 is gone; now on net PC13: CN7.13 (Pin_13)
- net PA14 is gone; now on net PC14: CN7.15 (Pin_15)
- net +3V3: now also CN7.18 (Pin_18); no longer CN7.12 (Pin_12), CN7.16 (Pin_16)
- net +5V: now also CN7.12 (Pin_12), CN7.16 (Pin_16); no longer CN7.18 (Pin_18)
- net AGND: now also Audio_In1.T, C1.2, C3.2, C5.2, C8.2, D1.1 (K), D2.1 (K), D3.1 (K), J1.2, J1.3, R12.1, R17.2, R18.2, R6.1, U3.4 (V-), U4.4 (V-), U6.4 (V-)
- net GND: now also U1.4 (V-), U2.4 (V-)
- net VIN: now also R11.2, R13.1, R16.2, R19.2, R5.2, SW1.2 (B), U1.7 (V+), U2.7 (V+), U3.7 (V+), U4.7 (V+), U6.7 (V+)
- net PA4 renamed DAC1
- net PC3 renamed ADC1
- net ADC1: now also R10.2, R11.1, R12.2, U3.3 (+), U4.3 (+); no longer CN7.35 (Pin_35)
- new net: C7.1, R4.1
- new net: C8.1, R5.1, R6.2, U6.3 (+)
- new net: R15.1, U3.6
- new net: D1.2 (A), R15.2
- new net: R16.1, R17.1, U4.2 (-)
- new net: R14.1, U4.6
- new net: C4.2, R8.2, R9.1
- new net: C5.1, R9.2, U2.3 (+)
- new net: D2.2 (A), R13.2
- new net: C6.2, R10.1
- new net: C2.1, R8.1, U1.2 (-), U1.6
- new net: C2.2, R2.2, R3.1
- new net: D3.2 (A), R14.2
- new net: R4.2, R7.2, U6.2 (-)
- new net: R18.1, R19.1, U3.2 (-)
- new net: C3.1, R3.2, U1.3 (+)
- new net: C4.1, C6.1, U2.2 (-), U2.6
- new net: J1.1, SW1.1 (A)
- new net: R1.1, R7.1, U6.6
- new net: C1.1, R1.2, R2.1
- new net Audio In: Audio_In1.S, C7.2
- new net PC2: CN7.35 (Pin_35)
- no-connect marks 8 -> 51
Other:
- note added: "9V Power Supply Barrel Connector"
- note added: "Audio In/Out"
- note added: "Audio Signal Conditioning"
- note added: "STM32 Shield"
- note added: "Volume Indicator"
- company: (none) -> Noisey Boyz
- title: (none) -> ANC on STM32
- moved on the sheet: CN10, CN11, CN5, CN6, CN8, CN9

Commit message: PCB routing finalized.
Parts:
- removed D1: LED, LED_THT:LED_D3.0mm, symbol Device:LED
- removed R12: 1K, Resistor_THT:R_Axial_DIN0204_L3.6mm_D1.6mm_P5.08mm_Horizontal, symbol Device:R
- removed R19: 220, Resistor_THT:R_Axial_DIN0204_L3.6mm_D1.6mm_P5.08mm_Horizontal, symbol Device:R
- removed U1, U2, U3, U4, U6: OP07, OP07DP:DIP794W45P254L959H508Q8, symbol Amplifier_Operational:OP07
- added C10: 10µ, Capacitor_THT:C_Axial_L3.8mm_D2.6mm_P7.50mm_Horizontal, symbol Device:C
- added C9: 100n, Capacitor_THT:C_Axial_L3.8mm_D2.6mm_P7.50mm_Horizontal, symbol Device:C
- added D2: LED, LED_THT:LED_D3.0mm, symbol Device:LED
- added LCD1: Conn_01x08, Connector_PinSocket_2.54mm:PinSocket_1x08_P2.54mm_Vertical, symbol Connector_Generic:Conn_01x08
- added R13: 23.3k, Resistor_THT:R_Axial_DIN0204_L3.6mm_D1.6mm_P5.08mm_Horizontal, symbol Device:R
- added RV1: R_Var, Potentiometer_THT:Potentiometer_ACP_CA9-H2,5_Horizontal, symbol Device:R_Potentiometer
- added U2: LM2903P, LM2903P:DIP794W45P254L959H508Q8, symbol LM2903P:LM2903P
- added U3: ~, custom_library:TL074, symbol custom_library:TL074
- C1: value 680p -> 150µ
- C3: value 220p -> 680p
- C4: value 1.8n -> 220p
- C5: value 180p -> 220p
- C6: value 270µ -> 680p
- C7: value 150µ -> 1.8n
- C8: value 1n -> 270µ
- R1: value 56K -> 31K
- R10: value 800 -> 4.45K
- R11: value 4.45K -> 1K
- R14: value 220 -> 17.7k
- R2: value 56K -> 1K
- R3: value 56K -> 150k
- R4: value 10K -> 56K
- R5: value 31K -> 56K
- R6: value 1K -> 56K
- R7: value 150k -> 56K
- R9: value 56K -> 800
- renumbered D2 to D1, R13 to R12
Connections:
- net +5V: now also LCD1.8 (Pin_8)
- net ADC1: now also R10.1, R11.2, R9.2, U2.3 (1IN+), U2.5 (2IN+); no longer R10.2, R11.1
- net AGND: now also C2.2, C4.2, C6.2, R11.1, R2.1, R7.1, D2.1 (K), RV1.3, U2.4 (GND), U3.11 (Vcc-), U3.6 (in_2_-), U3.7 (out_2); no longer C1.2, C8.2, R6.1
- net Audio In: now also C1.2; no longer C7.2
- net GND: now also C10.1, C9.1, LCD1.7 (Pin_7)
- net VIN: now also R1.2, R10.2, R14.2, C10.2, C9.2, R13.2, U2.8 (VCC), U3.4 (Vcc+); no longer R11.2, R16.2, R5.2
- net at R4.1: now also R3.1, U3.1 (out_1); no longer C7.1
- net at R15.1: now also U2.1 (1OUT)
- net at R15.2: now also D2.2 (A)
- net at R16.1: now also U2.7 (2OUT); no longer R17.1
- net at R14.1: now also R18.1, U2.6 (2IN-)
- net at C5.1: now also R6.2, U3.5 (in_2_+); no longer R9.2
- net at C2.1: now also R1.1, R2.2, U3.3 (in_1_+); no longer R8.1
- net at D3.2 (A): now also R16.2; no longer R14.2
- net at R4.2: now also C3.1, R5.1; no longer R7.2
- net at R3.2: now also RV1.2, U3.2 (in_1_-); no longer C3.1
- net at C4.1: now also R5.2, R6.1; no longer C6.1
- removed net +3V3: CN6.2 (Pin_2), CN6.4 (Pin_4), CN7.18 (Pin_18)
- net ARD D0 RX: no longer names the net of CN10.37 (Pin_37)
- net ARD D0 RX: no longer CN9.1 (Pin_1)
- net ARD D1 TX: no longer names the net of CN10.35 (Pin_35)
- net ARD D1 TX: no longer CN9.2 (Pin_2)
- net DAC1: no longer names the net of CN7.36 (Pin_36)
- net DAC1: no longer CN8.5 (Pin_5)
- net PA0: no longer names the net of CN7.28 (Pin_28)
- net PA0: no longer CN8.1 (Pin_1)
- net PA1: no longer names the net of CN7.30 (Pin_30)
- net PA1: no longer CN8.2 (Pin_2)
- net PA10: no longer names the net of CN10.33 (Pin_33)
- net PA10: no longer CN9.3 (Pin_3)
- net PA11: no longer names the net of CN10.14 (Pin_14)
- net PA12: no longer names the net of CN10.12 (Pin_12)
- net PA15: no longer names the net of CN7.17 (Pin_17)
- net PA2: no longer names the net of CN8.3 (Pin_3)
- net PA2: no longer CN7.32 (Pin_32)
- net PA3: no longer names the net of CN7.34 (Pin_34)
- net PA3: no longer CN8.4 (Pin_4)
- removed net PA5: CN10.11 (Pin_11), CN5.6 (Pin_6), CN7.38 (Pin_38), CN8.6 (Pin_6)
- net PA6: no longer names the net of CN10.13 (Pin_13)
- net PA6: no longer CN5.5 (Pin_5)
- net PA7: no longer names the net of CN5.4 (Pin_4)
- net PA7: no longer CN10.15 (Pin_15)
- net PA8: no longer names the net of CN10.23 (Pin_23)
- net PA8: no longer CN9.8 (Pin_8)
- net PA9: no longer names the net of CN10.21 (Pin_21)
- net PA9: no longer CN5.1 (Pin_1)
- net PB1: no longer names the net of CN10.24 (Pin_24)
- net PB10: no longer names the net of CN10.25 (Pin_25)
- net PB10: no longer CN9.7 (Pin_7)
- net PB11: no longer names the net of CN10.18 (Pin_18)
- net PB12: no longer names the net of CN10.16 (Pin_16)
- net PB13: no longer names the net of CN10.30 (Pin_30)
- net PB14: no longer names the net of CN10.28 (Pin_28)
- net PB15: no longer names the net of CN10.26 (Pin_26)
- net PB2: no longer names the net of CN10.22 (Pin_22)
- net PB3: no longer names the net of CN10.31 (Pin_31)
- net PB3: no longer CN9.4 (Pin_4)
- net PB4: no longer names the net of CN10.27 (Pin_27)
- net PB4: no longer CN9.6 (Pin_6)
- net PB5: no longer names the net of CN10.29 (Pin_29)
- net PB5: no longer CN9.5 (Pin_5)
- net PB6: no longer names the net of CN10.17 (Pin_17)
- net PB6: no longer CN5.3 (Pin_3)
- net PB7: no longer names the net of CN7.21 (Pin_21)
- removed net PB8: CN10.3 (Pin_3), CN5.10 (Pin_10), CN7.7 (Pin_7)
- net PB9: no longer names the net of CN10.5 (Pin_5)
- net PB9: no longer CN5.9 (Pin_9)
- net PC10: no longer names the net of CN7.1 (Pin_1)
- net PC11: no longer names the net of CN7.2 (Pin_2)
- net PC12: no longer names the net of CN7.3 (Pin_3)
- net PC13: no longer names the net of CN7.13 (Pin_13)
- net PC13: no longer CN7.23 (Pin_23)
- net PC14: no longer names the net of CN7.15 (Pin_15)
- net PC14: no longer CN7.25 (Pin_25)
- net PC15: no longer names the net of CN7.27 (Pin_27)
- net PC2: no longer names the net of CN7.35 (Pin_35)
- net PC4: no longer names the net of CN10.34 (Pin_34)
- net PC5: no longer names the net of CN10.6 (Pin_6)
- net PC6: no longer names the net of CN10.4 (Pin_4)
- net PC7: no longer names the net of CN10.19 (Pin_19)
- net PC7: no longer CN5.2 (Pin_2)
- net PC8: no longer names the net of CN10.2 (Pin_2)
- net PC9: no longer names the net of CN10.1 (Pin_1)
- net PD2: no longer names the net of CN7.4 (Pin_4)
- net PF0: no longer names the net of CN7.29 (Pin_29)
- net PF1: no longer names the net of CN7.31 (Pin_31)
- net T_NRST: no longer names the net of CN6.3 (Pin_3)
- net T_NRST: no longer CN7.14 (Pin_14)
- new net: C8.2, R9.1
- new net: C7.1, C8.1, U3.8 (out_3), U3.9 (in_3_-)
- new net: C1.1, RV1.1
- new net: R13.1, R17.1, U2.2 (1IN-)
- new net: C7.2, R7.2, R8.1
- new net: C6.1, R8.2, U3.10 (in_3_+)
- new net LCD_CS: CN8.5 (Pin_5), LCD1.4 (Pin_4)
- new net LCD_RS: CN8.1 (Pin_1), LCD1.6 (Pin_6)
- new net LCD_RST: CN8.2 (Pin_2), LCD1.5 (Pin_5)
- new net LED: CN8.4 (Pin_4), LCD1.1 (Pin_1)
- new net SCK: CN8.6 (Pin_6), LCD1.3 (Pin_3)
- new net SDI: CN10.15 (Pin_15), LCD1.2 (Pin_2)
- no-connect marks 51 -> 83
Other:
- note added: "LCD Display"
- moved on the sheet: Audio_In1

Commit message: PCB updated.
Parts:
- removed C1: 150µ, Capacitor_THT:C_Axial_L3.8mm_D2.6mm_P7.50mm_Horizontal, symbol Device:C
- removed C8: 270µ, Capacitor_THT:C_Axial_L3.8mm_D2.6mm_P7.50mm_Horizontal, symbol Device:C
- added C1: 150µ, Capacitor_THT:C_Radial_D4.0mm_H5.0mm_P1.50mm, symbol Device:C_Polarized
- added C8: 270µ, Capacitor_THT:C_Radial_D4.0mm_H5.0mm_P1.50mm, symbol Device:C_Polarized
- added H1, H2, H3, H4: MountingHole, MountingHole:MountingHole_3.2mm_M3_DIN965_Pad_TopBottom, symbol Mechanical:MountingHole
- added R19: 0, Resistor_THT:R_Axial_DIN0207_L6.3mm_D2.5mm_P7.62mm_Horizontal, symbol Device:R
- C10, C2, C3, C5, C7, C9: footprint Capacitor_THT:C_Axial_L3.8mm_D2.6mm_P7.50mm_Horizontal -> Capacitor_THT:C_Disc_D5.0mm_W2.5mm_P5.00mm
- C4: value 220p -> 1nF; footprint Capacitor_THT:C_Axial_L3.8mm_D2.6mm_P7.50mm_Horizontal -> Capacitor_THT:C_Disc_D5.0mm_W2.5mm_P5.00mm
- C6: value 680p -> 180p; footprint Capacitor_THT:C_Axial_L3.8mm_D2.6mm_P7.50mm_Horizontal -> Capacitor_THT:C_Disc_D5.0mm_W2.5mm_P5.00mm
- R1: value 31K -> 10k; footprint Resistor_THT:R_Axial_DIN0204_L3.6mm_D1.6mm_P5.08mm_Horizontal -> Resistor_THT:R_Axial_DIN0207_L6.3mm_D2.5mm_P7.62mm_Horizontal
- R10, R11, R13, R14, R17, R18, R3, R4, R5, R6, R7, R8, R9: footprint Resistor_THT:R_Axial_DIN0204_L3.6mm_D1.6mm_P5.08mm_Horizontal -> Resistor_THT:R_Axial_DIN0207_L6.3mm_D2.5mm_P7.62mm_Horizontal
- R12, R15, R16: value 220 -> 330; footprint Resistor_THT:R_Axial_DIN0204_L3.6mm_D1.6mm_P5.08mm_Horizontal -> Resistor_THT:R_Axial_DIN0207_L6.3mm_D2.5mm_P7.62mm_Horizontal
- R2: value 1K -> 10k; footprint Resistor_THT:R_Axial_DIN0204_L3.6mm_D1.6mm_P5.08mm_Horizontal -> Resistor_THT:R_Axial_DIN0207_L6.3mm_D2.5mm_P7.62mm_Horizontal
Connections:
- net +5V: now also LCD1.1 (Pin_1); no longer LCD1.8 (Pin_8)
- net AGND: now also C10.1, C9.1, R19.2
- net Audio In: now also C1.1
- net GND: now also LCD1.2 (Pin_2), R19.1; no longer C10.1, C9.1, LCD1.7 (Pin_7)
- net LCD_CS: now also CN8.3 (Pin_3), LCD1.3 (Pin_3); no longer CN8.5 (Pin_5), LCD1.4 (Pin_4)
- net LCD_RS: now also LCD1.5 (Pin_5); no longer LCD1.6 (Pin_6)
- net LCD_RST: now also LCD1.4 (Pin_4); no longer LCD1.5 (Pin_5)
- net LED: now also CN9.1 (Pin_1), LCD1.8 (Pin_8); no longer CN8.4 (Pin_4), LCD1.1 (Pin_1)
- net SCK: now also CN9.4 (Pin_4), LCD1.7 (Pin_7); no longer CN8.6 (Pin_6), LCD1.3 (Pin_3)
- net SDI: now also LCD1.6 (Pin_6); no longer LCD1.2 (Pin_2)
- net at R4.1, U3.1 (out_1): now also RV1.2; no longer R3.1
- net at R9.1: now also C8.2
- net at C7.1, U3.8 (out_3), U3.9 (in_3_-): now also C8.1
- net at RV1.1: now also R3.1, U3.2 (in_1_-)
- net +5V_USB_CHGR: no longer names the net of CN10.8 (Pin_8)
- net +5V_VIN: no longer names the net of CN6.1 (Pin_1)
- net +AREF: no longer names the net of CN5.8 (Pin_8)
- net +VREFP: no longer names the net of CN10.7 (Pin_7)
- net E5V: no longer names the net of CN7.6 (Pin_6)
- net VBAT: no longer names the net of CN7.33 (Pin_33)
- new net: C1.2, R3.2
- no-connect marks 83 -> 88
Other:
- note added: "Analog/Digital GND Bridge"
- note added: "Mounting Holes"

Commit message: PCB V1 Finalized
Parts:
- removed SW1: SW_SPST, Button_Switch_THT:SW_DIP_SPSTx01_Slide_9.78x4.72mm_W7.62mm_P2.54mm, symbol Switch:SW_SPST
- added S1: 100SP1T1B1M1QEH, 100SP1T1B1M1QEH:SW_100SP1T1B1M1QEH, symbol 100SP1T1B1M1QEH:100SP1T1B1M1QEH
Connections:
- net AGND: now also S1.1
- net VIN: now also S1.3
- net at J1.1: now also S1.2
Other:
- moved on the sheet: J1

Commit message: PCB board and firmware updated.
Parts:
- removed D3: LED, LED_THT:LED_D3.0mm, symbol Device:LED
- removed R16: 330, Resistor_THT:R_Axial_DIN0207_L6.3mm_D2.5mm_P7.62mm_Horizontal, symbol Device:R
- removed R17, R18: 10k, Resistor_THT:R_Axial_DIN0207_L6.3mm_D2.5mm_P7.62mm_Horizontal, symbol Device:R
- added C12: 10µ, Capacitor_THT:C_Disc_D5.0mm_W2.5mm_P5.00mm, symbol Device:C
- added C13: 1µ, Capacitor_THT:C_Disc_D5.0mm_W2.5mm_P5.00mm, symbol Device:C
- added C14: 0.1µ, Capacitor_THT:C_Radial_D4.0mm_H5.0mm_P1.50mm, symbol Device:C_Polarized
- added D4: D, Diode_THT:D_A-405_P7.62mm_Horizontal, symbol Device:D
- C1: value 150µ -> 10µ
- R13: value 23.3k -> 10k
- R14: value 17.7k -> 10k
- R15: value 330 -> 100
- R3: value 150k -> 10k
- R9: value 800 -> 50k
Connections:
- net +5V: now also R13.2, R15.2, U2.8 (VCC)
- net ADC1: now also C8.2, D4.2 (A); no longer R9.2, U2.3 (1IN+), U2.5 (2IN+)
- net AGND: now also C1.2, R14.1, R9.1, C12.1, C14.2; no longer C4.2, D2.1 (K), R7.1, U3.6 (in_2_-), U3.7 (out_2)
- net Audio In: now also C13.2; no longer C1.1
- net VIN: now also C12.2, C14.1; no longer R13.2, R14.2, U2.8 (VCC)
- net at R15.1: now also D2.2 (A); no longer U2.1 (1OUT)
- net at R3.2: now also C13.1; no longer C1.2
- net at U2.2 (1IN-): now also C1.1, R9.2, D4.1 (K); no longer R13.1
- net at U2.6 (2IN-): no longer R14.1
- new net: C4.2, R7.1, U3.6 (in_2_-), U3.7 (out_2)
- new net: D2.1 (K), U2.1 (1OUT)
- new net: R13.1, R14.2, U2.3 (1IN+)
- no-connect marks 88 -> 91
Other:
- moved on the sheet: D1, R10, R11, R12, U2
