File: PCB_Shield_STM32/PCB_Shield_STM32.kicad_pcb (KiCad board)
At the start: 2 copper layers, 100 x 100 mm, 46 parts, among them CN10 Conn_02x19_Odd_Even, CN11 Conn_01x02, CN12 Conn_01x02, CN5 Conn_01x10, CN6 Conn_01x08, CN7 Conn_02x19_Odd_Even, CN8 Conn_01x06, CN9 Conn_01x08, J1 Barrel_Jack_Switch, SW1 SW_SPST, U1 OP07, U2 OP07, U3 OP07, U4 OP07, U6 OP07

Commit message: PCB routing finalized.
Parts:
- removed the D1 at (118.5, 34.4)
- removed the R12 at (120.0, 57.2)
- removed R19: 220, Resistor_THT:R_Axial_DIN0204_L3.6mm_D1.6mm_P5.08mm_Horizontal
- removed U1, U4, U6: OP07, OP07DP:DIP794W45P254L959H508Q8
- added C10: 10µ, Capacitor_THT:C_Axial_L3.8mm_D2.6mm_P7.50mm_Horizontal, F.Cu at (94.1, 36.7)
- added C9: 100n, Capacitor_THT:C_Axial_L3.8mm_D2.6mm_P7.50mm_Horizontal, F.Cu at (94.1, 18.7)
- added D2: LED, LED_THT:LED_D3.0mm, F.Cu at (119.0, 81.6)
- added LCD1: Conn_01x08, Connector_PinSocket_2.54mm:PinSocket_1x08_P2.54mm_Vertical, F.Cu at (66.7, 108.8)
- added R13: 23.3k, Resistor_THT:R_Axial_DIN0204_L3.6mm_D1.6mm_P5.08mm_Horizontal, F.Cu at (97.1, 38.5)
- added RV1: R_Var, Potentiometer_THT:Potentiometer_ACP_CA9-H2,5_Horizontal, F.Cu at (113.2, 80.9)
- C1: value 680p -> 150µ
- C3: value 220p -> 680p
- C4: value 1.8n -> 220p
- C5: value 180p -> 220p
- C6: value 270µ -> 680p
- C7: value 150µ -> 1.8n
- C8: value 1n -> 270µ
- R1: value 56K -> 31K
- R10: value 800 -> 4.45K
- R11: value 4.45K -> 1K
- R14: value 220 -> 17.7k
- R2: value 56K -> 1K
- R3: value 56K -> 150k
- R4: value 10K -> 56K
- R5: value 31K -> 56K
- R6: value 1K -> 56K
- R7: value 150k -> 56K
- R9: value 56K -> 800
- U2: value OP07 -> LM2903P; footprint OP07DP:DIP794W45P254L959H508Q8 -> LM2903P:DIP794W45P254L959H508Q8
- U3: value OP07 -> ~; footprint OP07DP:DIP794W45P254L959H508Q8 -> custom_library:TL074
- moved SW1 114.6 mm to (41.2, 108.8)
- moved J1 99.6 mm to (36.5, 105.2), turned to 0 degrees
- moved CN7 98.5 mm to (89.0, 19.1), turned to 0 degrees
- moved CN12 96.4 mm to (88.9, 92.6), turned to 180 degrees
- moved CN11 95.9 mm to (25.5, 92.7), turned to 180 degrees
- moved R12 95.4 mm to (53.9, 106.9), turned to -90 degrees
- moved CN10 94.7 mm to (27.9, 19.1), turned to 0 degrees
- moved D1 90.8 mm to (59.8, 110.8), turned to 180 degrees
- moved CN9 88.2 mm to (33.5, 19.2), turned to 0 degrees
- moved C6 86.5 mm to (114.6, 24.1), turned to -90 degrees
- moved C8 84.3 mm to (114.6, 42.9), turned to 90 degrees
- moved R18 84.1 mm to (97.1, 29.3), turned to 90 degrees
- moved R11 69.8 mm to (105.9, 42.5), turned to -90 degrees
- moved CN8 66.2 mm to (80.4, 33.2), turned to 180 degrees
- moved R10 64.0 mm to (101.6, 47.6), turned to 90 degrees
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- renumbered CN12 to CN11, CN11 to CN12, D2 to D1, R13 to R12
Connections:
- C1 pad 2: AGND -> Audio In
- C2 pad 1: Net-(U1--) -> Net-(U3-in_1_+)
- C2 pad 2: Net-(C2-Pad2) -> AGND
- C3 pad 1: Net-(U1-+) -> Net-(C3-Pad1)
- C4 pad 1: Net-(U2--) -> Net-(C4-Pad1)
- C4 pad 2: Net-(C4-Pad2) -> AGND
- C5 pad 1: Net-(U2-+) -> Net-(U3-in_2_+)
- C6 pad 1: Net-(U2--) -> Net-(U3-in_3_+)
- C6 pad 2: Net-(C6-Pad2) -> AGND
- C7 pad 1: Net-(C7-Pad1) -> Net-(U3-in_3_-)
- C7 pad 2: Audio In -> Net-(C7-Pad2)
- C8 pad 1: Net-(U6-+) -> Net-(U3-in_3_-)
- C8 pad 2: AGND -> Net-(C8-Pad2)
- CN10 pad 1: /PC9 -> unconnected-(CN10-Pin_1-Pad1)
- CN10 pad 11: /PA5 -> unconnected-(CN10-Pin_11-Pad11)
- CN10 pad 12: /PA12 -> unconnected-(CN10-Pin_12-Pad12)
- CN10 pad 13: /PA6 -> unconnected-(CN10-Pin_13-Pad13)
- CN10 pad 14: /PA11 -> unconnected-(CN10-Pin_14-Pad14)
- CN10 pad 15: /PA7 -> /SDI
- CN10 pad 16: /PB12 -> unconnected-(CN10-Pin_16-Pad16)
- CN10 pad 17: /PB6 -> unconnected-(CN10-Pin_17-Pad17)
- CN10 pad 18: /PB11 -> unconnected-(CN10-Pin_18-Pad18)
- CN10 pad 19: /PC7 -> unconnected-(CN10-Pin_19-Pad19)
- CN10 pad 2: /PC8 -> unconnected-(CN10-Pin_2-Pad2)
- CN10 pad 21: /PA9 -> unconnected-(CN10-Pin_21-Pad21)
- CN10 pad 22: /PB2 -> unconnected-(CN10-Pin_22-Pad22)
- CN10 pad 23: /PA8 -> unconnected-(CN10-Pin_23-Pad23)
- CN10 pad 24: /PB1 -> unconnected-(CN10-Pin_24-Pad24)
- CN10 pad 25: /PB10 -> unconnected-(CN10-Pin_25-Pad25)
- CN10 pad 26: /PB15 -> unconnected-(CN10-Pin_26-Pad26)
- CN10 pad 27: /PB4 -> unconnected-(CN10-Pin_27-Pad27)
- CN10 pad 28: /PB14 -> unconnected-(CN10-Pin_28-Pad28)
- CN10 pad 29: /PB5 -> unconnected-(CN10-Pin_29-Pad29)
- CN10 pad 3: /PB8 -> unconnected-(CN10-Pin_3-Pad3)
- CN10 pad 30: /PB13 -> unconnected-(CN10-Pin_30-Pad30)
- CN10 pad 31: /PB3 -> unconnected-(CN10-Pin_31-Pad31)
- CN10 pad 33: /PA10 -> unconnected-(CN10-Pin_33-Pad33)
- CN10 pad 34: /PC4 -> unconnected-(CN10-Pin_34-Pad34)
- CN10 pad 35: /ARD D1 TX -> unconnected-(CN10-Pin_35-Pad35)
- CN10 pad 37: /ARD D0 RX -> unconnected-(CN10-Pin_37-Pad37)
- CN10 pad 4: /PC6 -> unconnected-(CN10-Pin_4-Pad4)
- CN10 pad 5: /PB9 -> unconnected-(CN10-Pin_5-Pad5)
- CN10 pad 6: /PC5 -> unconnected-(CN10-Pin_6-Pad6)
- CN5 pad 1: /PA9 -> unconnected-(CN5-Pin_1-Pad1)
- CN5 pad 10: /PB8 -> unconnected-(CN5-Pin_10-Pad10)
- CN5 pad 2: /PC7 -> unconnected-(CN5-Pin_2-Pad2)
- CN5 pad 3: /PB6 -> unconnected-(CN5-Pin_3-Pad3)
- CN5 pad 4: /PA7 -> unconnected-(CN5-Pin_4-Pad4)
- CN5 pad 5: /PA6 -> unconnected-(CN5-Pin_5-Pad5)
- CN5 pad 6: /PA5 -> unconnected-(CN5-Pin_6-Pad6)
- CN5 pad 9: /PB9 -> unconnected-(CN5-Pin_9-Pad9)
- CN6 pad 2: +3V3 -> unconnected-(CN6-Pin_2-Pad2)
- CN6 pad 3: /T_NRST -> unconnected-(CN6-Pin_3-Pad3)
- CN6 pad 4: +3V3 -> unconnected-(CN6-Pin_4-Pad4)
- CN7 pad 1: /PC10 -> unconnected-(CN7-Pin_1-Pad1)
- CN7 pad 13: /PC13 -> unconnected-(CN7-Pin_13-Pad13)
- CN7 pad 14: /T_NRST -> unconnected-(CN7-Pin_14-Pad14)
- CN7 pad 15: /PC14 -> unconnected-(CN7-Pin_15-Pad15)
- CN7 pad 17: /PA15 -> unconnected-(CN7-Pin_17-Pad17)
- CN7 pad 18: +3V3 -> unconnected-(CN7-Pin_18-Pad18)
- CN7 pad 2: /PC11 -> unconnected-(CN7-Pin_2-Pad2)
- CN7 pad 21: /PB7 -> unconnected-(CN7-Pin_21-Pad21)
- CN7 pad 23: /PC13 -> unconnected-(CN7-Pin_23-Pad23)
- CN7 pad 25: /PC14 -> unconnected-(CN7-Pin_25-Pad25)
- CN7 pad 27: /PC15 -> unconnected-(CN7-Pin_27-Pad27)
- CN7 pad 28: /PA0 -> unconnected-(CN7-Pin_28-Pad28)
- CN7 pad 29: /PF0 -> unconnected-(CN7-Pin_29-Pad29)
- CN7 pad 3: /PC12 -> unconnected-(CN7-Pin_3-Pad3)
- CN7 pad 30: /PA1 -> unconnected-(CN7-Pin_30-Pad30)
- CN7 pad 31: /PF1 -> unconnected-(CN7-Pin_31-Pad31)
- CN7 pad 32: /PA2 -> unconnected-(CN7-Pin_32-Pad32)
- CN7 pad 34: /PA3 -> unconnected-(CN7-Pin_34-Pad34)
- CN7 pad 35: /PC2 -> unconnected-(CN7-Pin_35-Pad35)
- CN7 pad 36: /DAC1 -> unconnected-(CN7-Pin_36-Pad36)
- CN7 pad 38: /PA5 -> unconnected-(CN7-Pin_38-Pad38)
- CN7 pad 4: /PD2 -> unconnected-(CN7-Pin_4-Pad4)
- CN7 pad 7: /PB8 -> unconnected-(CN7-Pin_7-Pad7)
- CN8 pad 1: /PA0 -> /LCD_RS
- CN8 pad 2: /PA1 -> /LCD_RST
- CN8 pad 3: /PA2 -> unconnected-(CN8-Pin_3-Pad3)
- CN8 pad 4: /PA3 -> /LED
- CN8 pad 5: /DAC1 -> /LCD_CS
- CN8 pad 6: /PA5 -> /SCK
- CN9 pad 1: /ARD D0 RX -> unconnected-(CN9-Pin_1-Pad1)
- CN9 pad 2: /ARD D1 TX -> unconnected-(CN9-Pin_2-Pad2)
- CN9 pad 3: /PA10 -> unconnected-(CN9-Pin_3-Pad3)
- CN9 pad 4: /PB3 -> unconnected-(CN9-Pin_4-Pad4)
- CN9 pad 5: /PB5 -> unconnected-(CN9-Pin_5-Pad5)
- CN9 pad 6: /PB4 -> unconnected-(CN9-Pin_6-Pad6)
- CN9 pad 7: /PB10 -> unconnected-(CN9-Pin_7-Pad7)
- CN9 pad 8: /PA8 -> unconnected-(CN9-Pin_8-Pad8)
- R1 pad 1: Net-(R1-Pad1) -> Net-(U3-in_1_+)
- R1 pad 2: Net-(C1-Pad1) -> VIN
- R10 pad 1: Net-(C6-Pad2) -> ADC1
- R10 pad 2: ADC1 -> VIN
- R11 pad 1: ADC1 -> AGND
- R11 pad 2: VIN -> ADC1
- R14 pad 1: Net-(R14-Pad1) -> Net-(U2-2IN-)
- R14 pad 2: Net-(D3-A) -> VIN
- R15 pad 1: Net-(R15-Pad1) -> Net-(U2-1OUT)
- R16 pad 1: Net-(U4--) -> Net-(U2-2OUT)
- R16 pad 2: VIN -> Net-(D3-A)
- R17 pad 1: Net-(U4--) -> Net-(U2-1IN-)
- R18 pad 1: Net-(U3--) -> Net-(U2-2IN-)
- R2 pad 1: Net-(C1-Pad1) -> AGND
- R2 pad 2: Net-(C2-Pad2) -> Net-(U3-in_1_+)
- R3 pad 1: Net-(C2-Pad2) -> Net-(U3-out_1)
- R3 pad 2: Net-(U1-+) -> Net-(U3-in_1_-)
- R4 pad 1: Net-(C7-Pad1) -> Net-(U3-out_1)
- R4 pad 2: Net-(U6--) -> Net-(C3-Pad1)
- R5 pad 1: Net-(U6-+) -> Net-(C3-Pad1)
- R5 pad 2: VIN -> Net-(C4-Pad1)
- R6 pad 1: AGND -> Net-(C4-Pad1)
- R6 pad 2: Net-(U6-+) -> Net-(U3-in_2_+)
- R7 pad 1: Net-(R1-Pad1) -> AGND
- R7 pad 2: Net-(U6--) -> Net-(C7-Pad2)
- R8 pad 1: Net-(U1--) -> Net-(C7-Pad2)
- R8 pad 2: Net-(C4-Pad2) -> Net-(U3-in_3_+)
- R9 pad 1: Net-(C4-Pad2) -> Net-(C8-Pad2)
- R9 pad 2: Net-(U2-+) -> ADC1
- U2 pad 1: unconnected-(U2-VOS-Pad1) -> Net-(U2-1OUT)
- U2 pad 2: Net-(U2--) -> Net-(U2-1IN-)
- U2 pad 3: Net-(U2-+) -> ADC1
- U2 pad 4: GND -> AGND
- U2 pad 5: unconnected-(U2-NC-Pad5) -> ADC1
- U2 pad 6: Net-(U2--) -> Net-(U2-2IN-)
- U2 pad 7: VIN -> Net-(U2-2OUT)
- U2 pad 8: unconnected-(U2-VOS-Pad8) -> VIN
- U3 pad 1: unconnected-(U3-VOS-Pad1) -> Net-(U3-out_1)
- U3 pad 2: Net-(U3--) -> Net-(U3-in_1_-)
- U3 pad 3: ADC1 -> Net-(U3-in_1_+)
- U3 pad 4: AGND -> VIN
- U3 pad 5: unconnected-(U3-NC-Pad5) -> Net-(U3-in_2_+)
- U3 pad 6: Net-(R15-Pad1) -> AGND
- U3 pad 7: VIN -> AGND
- U3 pad 8: unconnected-(U3-VOS-Pad8) -> Net-(U3-in_3_-)
Routing:
- net AGND: track 26.2 -> 374.4 mm, vias 0 -> 6
- net GND: track 1.67 -> 249.6 mm, vias 0 -> 2
- net /LED: track 0.00 -> 113.2 mm
- net Net-(U3-in_2_+): track 0.00 -> 113.2 mm, vias 0 -> 2
- net /SCK: track 0.00 -> 101.0 mm
- net /SDI: track 0.00 -> 98.8 mm
- net /LCD_CS: track 0.00 -> 98.1 mm
- net /LCD_RST: track 0.00 -> 89.9 mm
- net /LCD_RS: track 0.00 -> 84.9 mm
- net Net-(U3-in_3_+): track 0.00 -> 81.7 mm, vias 0 -> 6
- net +5V: track 0.00 -> 74.0 mm
- net Net-(U3-in_3_-): track 0.00 -> 71.7 mm, vias 0 -> 2
- net Net-(U3-in_1_+): track 0.00 -> 68.2 mm, vias 0 -> 3
- net VIN: track 141.7 -> 207.8 mm, vias 0 -> 5
- net Net-(U2-2IN-): track 0.00 -> 58.3 mm
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
Commit message: PCB updated.
Parts:
- added H1: MountingHole, MountingHole:MountingHole_3.2mm_M3_DIN965_Pad_TopBottom, F.Cu at (45.4, 100.1)
- added H2: MountingHole, MountingHole:MountingHole_3.2mm_M3_DIN965_Pad_TopBottom, F.Cu at (117.7, 19.6)
- added H3: MountingHole, MountingHole:MountingHole_3.2mm_M3_DIN965_Pad_TopBottom, F.Cu at (45.3, 29.6)
- added H4: MountingHole, MountingHole:MountingHole_3.2mm_M3_DIN965_Pad_TopBottom, F.Cu at (110.4, 91.7)
- added R19: 0, Resistor_THT:R_Axial_DIN0207_L6.3mm_D2.5mm_P7.62mm_Horizontal, F.Cu at (25.3, 97.8)
- C1, C8: footprint Capacitor_THT:C_Axial_L3.8mm_D2.6mm_P7.50mm_Horizontal -> Capacitor_THT:C_Radial_D4.0mm_H5.0mm_P1.50mm
- C10, C2, C3, C5, C7, C9: footprint Capacitor_THT:C_Axial_L3.8mm_D2.6mm_P7.50mm_Horizontal -> Capacitor_THT:C_Disc_D5.0mm_W2.5mm_P5.00mm
- C4: value 220p -> 1nF; footprint Capacitor_THT:C_Axial_L3.8mm_D2.6mm_P7.50mm_Horizontal -> Capacitor_THT:C_Disc_D5.0mm_W2.5mm_P5.00mm
- C6: value 680p -> 180p; footprint Capacitor_THT:C_Axial_L3.8mm_D2.6mm_P7.50mm_Horizontal -> Capacitor_THT:C_Disc_D5.0mm_W2.5mm_P5.00mm
- R1: value 31K -> 10k; footprint Resistor_THT:R_Axial_DIN0204_L3.6mm_D1.6mm_P5.08mm_Horizontal -> Resistor_THT:R_Axial_DIN0207_L6.3mm_D2.5mm_P7.62mm_Horizontal
- R10, R11, R13, R14, R17, R18, R3, R4, R5, R6, R7, R8, R9: footprint Resistor_THT:R_Axial_DIN0204_L3.6mm_D1.6mm_P5.08mm_Horizontal -> Resistor_THT:R_Axial_DIN0207_L6.3mm_D2.5mm_P7.62mm_Horizontal
- R12, R15, R16: value 220 -> 330; footprint Resistor_THT:R_Axial_DIN0204_L3.6mm_D1.6mm_P5.08mm_Horizontal -> Resistor_THT:R_Axial_DIN0207_L6.3mm_D2.5mm_P7.62mm_Horizontal
- R2: value 1K -> 10k; footprint Resistor_THT:R_Axial_DIN0204_L3.6mm_D1.6mm_P5.08mm_Horizontal -> Resistor_THT:R_Axial_DIN0207_L6.3mm_D2.5mm_P7.62mm_Horizontal
- moved LCD1 17.3 mm to (84.1, 108.5), turned to -90 degrees
- moved C1 11.9 mm to (118.0, 97.8), turned to 180 degrees
- moved CN6 7.35 mm to (81.3, 54.8)
- moved C4 6.63 mm to (120.5, 36.2), turned to 180 degrees
- moved R5 6.52 mm to (104.0, 18.3)
- moved C9 5.58 mm to (95.3, 24.1)
- moved C5 5.27 mm to (115.3, 93.9)
- moved C8 4.35 mm to (118.7, 41.6), turned to 180 degrees
- moved R18 4.32 mm to (99.7, 25.9)
- moved R6 4.32 mm to (108.6, 25.9)
- moved R10 2.92 mm to (104.2, 48.9)
- moved R11 2.91 mm to (108.6, 41.3)
- moved R13 2.91 mm to (99.7, 37.2)
- moved R14 2.91 mm to (104.1, 37.2)
- moved R17 2.91 mm to (108.5, 37.2)
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Connections:
- C1 pad 1: Net-(C1-Pad1) -> Audio In
- C1 pad 2: Audio In -> Net-(C1-Pad2)
- C10 pad 1: GND -> AGND
- C9 pad 1: GND -> AGND
- CN10 pad 7: +VREFP -> unconnected-(CN10-Pin_7-Pad7)
- CN10 pad 8: +5V_USB_CHGR -> unconnected-(CN10-Pin_8-Pad8)
- CN5 pad 8: +AREF -> unconnected-(CN5-Pin_8-Pad8)
- CN6 pad 1: +5V_VIN -> unconnected-(CN6-Pin_1-Pad1)
- CN7 pad 33: VBAT -> unconnected-(CN7-Pin_33-Pad33)
- CN7 pad 6: E5V -> unconnected-(CN7-Pin_6-Pad6)
- CN8 pad 3: unconnected-(CN8-Pin_3-Pad3) -> /LCD_CS
- CN8 pad 4: /LED -> unconnected-(CN8-Pin_4-Pad4)
- CN8 pad 5: /LCD_CS -> unconnected-(CN8-Pin_5-Pad5)
- CN8 pad 6: /SCK -> unconnected-(CN8-Pin_6-Pad6)
- CN9 pad 1: unconnected-(CN9-Pin_1-Pad1) -> /LED
- CN9 pad 4: unconnected-(CN9-Pin_4-Pad4) -> /SCK
- LCD1 pad 1: /LED -> +5V
- LCD1 pad 2: /SDI -> GND
- LCD1 pad 3: /SCK -> /LCD_CS
- LCD1 pad 4: /LCD_CS -> /LCD_RST
- LCD1 pad 5: /LCD_RST -> /LCD_RS
- LCD1 pad 6: /LCD_RS -> /SDI
- LCD1 pad 7: GND -> /SCK
- LCD1 pad 8: +5V -> /LED
- R3 pad 1: Net-(U3-out_1) -> Net-(U3-in_1_-)
- R3 pad 2: Net-(U3-in_1_-) -> Net-(C1-Pad2)
- RV1 pad 1: Net-(C1-Pad1) -> Net-(U3-in_1_-)
- RV1 pad 2: Net-(U3-in_1_-) -> Net-(U3-out_1)
Routing:
- net GND: track 249.6 -> 213.6 mm, vias 2 -> 0
- net Net-(C1-Pad2): track 0.00 -> 28.4 mm, vias 0 -> 1
- net Net-(U3-in_1_-): track 31.3 -> 58.2 mm, vias 0 -> 1
- net /SDI: track 98.8 -> 108.4 mm
- net VIN: track 207.8 -> 198.8 mm, vias 5 -> 4
- net Net-(U3-in_2_+): track 113.2 -> 121.1 mm
- net +5V: track 74.0 -> 81.9 mm
- net Net-(C4-Pad1): track 33.2 -> 25.7 mm
- net Net-(C1-Pad1): track 6.17 -> 0.00 mm
- net /LED: track 113.2 -> 107.7 mm
- net AGND: track 374.4 -> 369.0 mm, vias 6 -> 2
- net Net-(U3-in_1_+): track 68.2 -> 73.4 mm, vias 3 -> 1
- net Net-(C7-Pad2): track 13.3 -> 18.3 mm
- net Net-(C3-Pad1): track 54.7 -> 50.1 mm, vias 2 -> 0
- net Net-(U3-in_3_+): track 81.7 -> 85.3 mm, vias 6 -> 2
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
Commit message: PCB V1 Finalized
Parts:
- removed SW1: SW_SPST, Button_Switch_THT:SW_DIP_SPSTx01_Slide_9.78x4.72mm_W7.62mm_P2.54mm
- added S1: 100SP1T1B1M1QEH, 100SP1T1B1M1QEH:SW_100SP1T1B1M1QEH, F.Cu at (44.9, 103.0)
- moved H1 13.9 mm to (40.1, 87.3)
- moved R12 4.45 mm to (52.0, 102.8)
- moved H4 0.45 mm to (110.1, 91.3)
- moved CN5 0.09 mm to (33.1, 41.5)
- moved CN9 0.09 mm to (33.1, 19.1)
Routing:
- net AGND: track 369.0 -> 381.3 mm, vias 2 -> 4
- net Net-(J1-Pad1): track 7.33 -> 9.79 mm
- net VIN: track 198.8 -> 199.7 mm
- net Net-(D1-A): track 5.11 -> 5.72 mm
- added copper zone on B.Cu, net AGND
- added copper zone on F.Cu, net AGND

Commit message: PCB board and firmware updated.
Parts:
- removed D3: LED, LED_THT:LED_D3.0mm
- removed R16: 330, Resistor_THT:R_Axial_DIN0207_L6.3mm_D2.5mm_P7.62mm_Horizontal
- removed R17, R18: 10k, Resistor_THT:R_Axial_DIN0207_L6.3mm_D2.5mm_P7.62mm_Horizontal
- added C12: 10µ, Capacitor_THT:C_Disc_D5.0mm_W2.5mm_P5.00mm, F.Cu at (39.1, 109.4)
- added C13: 1µ, Capacitor_THT:C_Disc_D5.0mm_W2.5mm_P5.00mm, F.Cu at (113.9, 53.9)
- added C14: 0.1µ, Capacitor_THT:C_Radial_D4.0mm_H5.0mm_P1.50mm, F.Cu at (44.7, 106.4)
- added D4: D, Diode_THT:D_A-405_P7.62mm_Horizontal, F.Cu at (107.9, 29.3)
- C1: value 150µ -> 10µ
- R13: value 23.3k -> 10k
- R14: value 17.7k -> 10k
- R15: value 330 -> 100
- R3: value 150k -> 10k
- R9: value 800 -> 50k
- moved R5 71.5 mm to (96.1, 89.3)
- moved R6 71.4 mm to (110.7, 97.3)
- moved C1 69.0 mm to (118.9, 28.9), turned to 90 degrees
- moved D2 44.2 mm to (118.9, 37.4)
- moved D1 43.3 mm to (24.6, 85.4), turned to 90 degrees
- moved C2 42.2 mm to (105.5, 54.1), turned to -90 degrees
- moved R4 39.9 mm to (101.0, 97.0)
- moved C3 39.9 mm to (100.1, 59.1), turned to 90 degrees
- moved C5 35.4 mm to (109.7, 59.0)
- moved C7 35.0 mm to (107.8, 23.7), turned to 90 degrees
- moved S1 34.0 mm to (26.2, 74.5)
- moved C4 33.9 mm to (95.5, 59.1), turned to 90 degrees
- moved R13 33.8 mm to (95.7, 70.8)
- moved U2 33.6 mm to (99.2, 33.2), turned to 90 degrees
- moved R3 28.8 mm to (105.8, 89.7)
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Connections:
- C1 pad 1: Audio In -> Net-(D4-K)
- C1 pad 2: Net-(C1-Pad2) -> AGND
- C4 pad 2: AGND -> Net-(U3-in_2_-)
- C8 pad 2: Net-(C8-Pad2) -> ADC1
- D2 pad 1: AGND -> Net-(D2-K)
- R13 pad 1: Net-(U2-1IN-) -> Net-(U2-1IN+)
- R13 pad 2: VIN -> +5V
- R14 pad 1: Net-(U2-2IN-) -> AGND
- R14 pad 2: VIN -> Net-(U2-1IN+)
- R15 pad 1: Net-(U2-1OUT) -> Net-(D2-A)
- R15 pad 2: Net-(D2-A) -> +5V
- R3 pad 2: Net-(C1-Pad2) -> Net-(C13-Pad1)
- R7 pad 1: AGND -> Net-(U3-in_2_-)
- R9 pad 1: Net-(C8-Pad2) -> AGND
- R9 pad 2: ADC1 -> Net-(D4-K)
- U2 pad 1: Net-(U2-1OUT) -> Net-(D2-K)
- U2 pad 2: Net-(U2-1IN-) -> Net-(D4-K)
- U2 pad 3: ADC1 -> Net-(U2-1IN+)
- U2 pad 5: ADC1 -> unconnected-(U2-2IN+-Pad5)
- U2 pad 6: Net-(U2-2IN-) -> unconnected-(U2-2IN--Pad6)
- U2 pad 7: Net-(U2-2OUT) -> unconnected-(U2-2OUT-Pad7)
- U2 pad 8: VIN -> +5V
- U3 pad 6: AGND -> Net-(U3-in_2_-)
- U3 pad 7: AGND -> Net-(U3-in_2_-)
Routing:
- net AGND: track 381.3 -> 46.4 mm, vias 4 -> 3
- net VIN: track 199.7 -> 318.9 mm, vias 4 -> 3
- net Net-(U3-in_2_+): track 121.1 -> 32.9 mm, vias 2 -> 0
- net +5V: track 81.9 -> 156.4 mm
- net Net-(C13-Pad1): track 0.00 -> 67.3 mm
- net Net-(U2-2IN-): track 59.2 -> 0.00 mm, vias 2 -> 0
- net Net-(U2-1IN+): track 0.00 -> 53.9 mm
- net Net-(D4-K): track 0.00 -> 53.8 mm
- net Net-(C7-Pad2): track 18.3 -> 68.4 mm, vias 0 -> 1
- net Net-(U2-2OUT): track 48.5 -> 0.00 mm
- net Net-(U2-1IN-): track 41.8 -> 0.00 mm
- net Net-(U3-in_2_-): track 0.00 -> 40.2 mm
- net Audio In: track 11.3 -> 51.2 mm
- net Net-(U3-in_1_-): track 58.2 -> 19.4 mm, vias 1 -> 0
- net Net-(D2-K): track 0.00 -> 29.7 mm, vias 0 -> 1
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- removed copper zone on B.Cu, net AGND
- removed copper zone on F.Cu, net AGND
Other:
- board text added: "9VDC"
- board text added: "LCD"

Commit message: Added latest firmware.
Parts:
- moved H3 27.1 mm to (20.3, 18.9)
- moved H4 22.8 mm to (95.5, 110.2)
- moved J1 7.42 mm to (25.9, 103.3)
- moved D1 6.78 mm to (18.6, 82.4), turned to -90 degrees
- moved S1 6.70 mm to (19.9, 72.1)
- moved Audio_In1 6.41 mm to (117.5, 106.2)
- moved CN12 6.41 mm to (95.1, 88.4)
- moved R13 6.41 mm to (101.9, 69.1)
- moved R3 6.41 mm to (112.0, 87.9)
- moved R7 6.41 mm to (116.7, 69.1)
- moved U3 6.41 mm to (101.0, 83.9)
- moved C1 6.41 mm to (125.1, 27.2)
- moved C10 6.41 mm to (109.6, 16.9)
- moved C3 6.41 mm to (106.3, 57.4)
- moved C6 6.41 mm to (105.4, 21.9)
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Routing:
- net VIN: track 318.9 -> 342.4 mm
- net Net-(J1-Pad1): track 37.3 -> 58.9 mm
- net AGND: track 46.4 -> 42.5 mm
- net GND: track 214.9 -> 211.3 mm
- net Net-(D1-A): track 7.07 -> 5.86 mm
- added copper zone on B.Cu, net AGND
- added copper zone on F.Cu, net AGND
Other:
- board size 100 x 100 mm -> 112.7 x 100 mm
